File: cad/schema_analog_digital/pressuremon.kicad_pcb (KiCad board)
At the start: 2 copper layers, 70 x 50 mm, 19 parts, among them J1 Digital Pressure 1, J2 Digital Pressure 2, J3 Analog Pressure 1, J4 Analog Pressure 2, Q1 BC337, U3 DS18B20

Commit message: Update analog pcb
Parts:
- removed ? (x3): , 
- removed JP1: SolderJumper_2_Open, Jumper:SolderJumper-2_P1.3mm_Open_RoundedPad1.0x1.5mm
- removed Q1: BC337, Package_TO_SOT_THT:TO-92S_Wide
- removed R6: 1k, Resistor_THT:R_Axial_DIN0204_L3.6mm_D1.6mm_P7.62mm_Horizontal
- removed REF**: MountingHole_2.2mm_M2, MountingHole:MountingHole_2.2mm_M2
- removed U2: ~, pressuremon_library:adc1115
- added H1: MountingHole_Pad, MountingHole:MountingHole_2.2mm_M2_ISO7380_Pad, F.Cu at (110.6, 43.0)
- added H2: MountingHole_Pad, MountingHole:MountingHole_2.2mm_M2_ISO7380_Pad, F.Cu at (175.6, 42.8)
- added H3: MountingHole_Pad, MountingHole:MountingHole_2.2mm_M2_ISO7380_Pad, F.Cu at (175.6, 88.2)
- added H4: MountingHole_Pad, MountingHole:MountingHole_2.2mm_M2_ISO7380_Pad, F.Cu at (110.4, 88.2)
- added J5: Conn_01x03_Pin, Connector_PinHeader_2.54mm:PinHeader_1x03_P2.54mm_Vertical, F.Cu at (168.2, 56.8)
- added SW1: SW_DPDT_x2, Connector_PinHeader_2.54mm:PinHeader_1x03_P2.54mm_Vertical, F.Cu at (168.4, 66.7)
- added U4: ~, pressuremon_library:ads1115, F.Cu at (113.0, 51.3)
- U3: footprint Package_TO_SOT_THT:TO-92_Inline_Wide -> Package_TO_SOT_THT:TO-92L_Inline_Wide
- moved R5 29.2 mm to (135.4, 79.2), turned to 0 degrees
- moved J1 22.8 mm to (168.9, 85.0), turned to -90 degrees
- moved R4 19.1 mm to (153.4, 79.2), turned to 180 degrees
- moved R3 19.1 mm to (156.2, 79.2), turned to 0 degrees
- moved J2 18.1 mm to (151.7, 85.0), turned to -90 degrees
- moved R2 17.0 mm to (174.0, 79.2), turned to 180 degrees
- moved U1 7.47 mm to (134.6, 51.5)
- moved J3 4.52 mm to (132.9, 85.0)
- moved J4 3.50 mm to (120.2, 85.0)
- moved U3 2.02 mm to (114.1, 46.0)
- moved R1 0.78 mm to (125.0, 46.0)
Connections:
- U1 pad 1: +3.3V -> unconnected-(U1-3.3V-Pad1)
- U1 pad 10: GND -> Net-(J5-Pin_3)
- U1 pad 11: unconnected-(U1-6-Pad11) -> /SCL
- U1 pad 12: unconnected-(U1-7(LED)-Pad12) -> /SDA
- U1 pad 13: /SDA -> unconnected-(U1-7(LED)-Pad13)
- U1 pad 14: /SCL -> unconnected-(U1-6-Pad14)
- U1 pad 15: unconnected-(U1-RX-Pad15) -> GND
- U1 pad 16: unconnected-(U1-TX-Pad16) -> +5V
- U1 pad 3: Net-(U1-4(MOSI)) -> /VCC
- U1 pad 8: unconnected-(U1-EN/RST-Pad8) -> Net-(SW1A-C)
- U1 pad 9: +5V -> Net-(J5-Pin_2)
Routing:
- net +3.3V: track 60.0 -> 0.00 mm
- net /VCC: track 148.2 -> 200.0 mm
- net Net-(J5-Pin_2): track 0.00 -> 44.2 mm
- net Net-(J5-Pin_3): track 0.00 -> 42.7 mm
- net Net-(U1-4(MOSI)): track 34.3 -> 0.00 mm
- net /SCL: track 83.4 -> 56.6 mm
- net /SDA: track 75.6 -> 54.4 mm
- net /SCL1: track 45.9 -> 30.6 mm
- net Net-(U1-5): track 33.9 -> 46.6 mm
- net Net-(SW1A-C): track 0.00 -> 12.0 mm
- net Net-(Q1-B): track 5.99 -> 0.00 mm
- net /DATA1: track 15.7 -> 20.6 mm
- net /DATA: track 19.5 -> 20.9 mm
- net /SDA1: track 58.1 -> 56.8 mm
- net unconnected-(U1-6-Pad11): track 0.62 -> 0.00 mm
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Other:
- board text added: "Pressuremon v1.3 ESP32 C3 PICO, Digital and Analog (c) 2025 Magnus Persson"
- board text removed: "Pressuremon v1.0 ESP32 C3 PICO, Digital and Analog (c) 2025 Magnus Persson"
