File: cad/schema_analog_digital/pressuremon-backups/pressuremon-2025-03-26_163811/pressuremon.kicad_sch (KiCad schematic)
At the start: 18 parts, among them J1 Digital Pressure 1, J2 Digital Pressure 2, J3 Analog Pressure 1, J4 Analog Pressure 2, J5 Conn_01x03_Pin, SW1 SW_DPDT_x2, U3 DS18B20

Commit message: Update analog pcb
Parts:
- removed H1, H2, H3, H4: MountingHole_Pad, MountingHole:MountingHole_2.2mm_M2_ISO7380_Pad, symbol Mechanical:MountingHole_Pad
- removed J5: Conn_01x03_Pin, Connector_PinHeader_2.54mm:PinHeader_1x03_P2.54mm_Vertical, symbol Connector:Conn_01x03_Pin
- removed SW1: SW_DPDT_x2, Connector_PinHeader_2.54mm:PinHeader_1x03_P2.54mm_Vertical, symbol Switch:SW_DPDT_x2
- removed U1: ~, pressuremon_library:ESP32C3-pico, symbol esp32c3-pico:ESP32C3-pico
- removed U4: ~, pressuremon_library:ads1115, symbol ads1115:ADS1115
- added JP1: SolderJumper_2_Open, Jumper:SolderJumper-2_P1.3mm_Open_RoundedPad1.0x1.5mm, symbol Jumper:SolderJumper_2_Open
- added Q1: BC337, Package_TO_SOT_THT:TO-92S_Wide, symbol Transistor_BJT:BC337
- added R6: 1k, Resistor_THT:R_Axial_DIN0204_L3.6mm_D1.6mm_P7.62mm_Horizontal, symbol Device:R
- added U1: ~, pressuremon_library:ESP32C3-pico, symbol myCommonSymbols:ESP32C3-pico
- added U2: ~, pressuremon_library:adc1115, symbol pressuremon_library:ADS1115
- U3: footprint Package_TO_SOT_THT:TO-92L_Inline_Wide -> Package_TO_SOT_THT:TO-92_Inline_Wide
Connections:
- net +5V: now also U1.9 (5V)
- net DATA: now also U2.7 (A0)
- net DATA1: now also U2.8 (A1)
- net GND: now also U1.10 (GND), U1.4 (0(MISO)), U2.10 (A3), U2.2 (GND), U2.5 (ADDR), U2.9 (A2)
- net SCL: now also U1.14 (10(SCL)), U2.3 (SCL)
- net SCL1: now also U1.6 (2)
- net SDA: now also U1.13 (8(SDA)), U2.4 (SDA)
- net SDA1: now also U1.5 (1(SCK))
- net VCC: now also JP1.1 (A), Q1.3 (E), U2.1 (VDD)
- net at R1.2, U3.2 (DQ): now also U1.2 (5)
- new net: R6.1, U1.3 (4(MOSI))
- new net: Q1.2 (B), R6.2
- new net +3.3V: JP1.2 (B), Q1.1 (C), U1.1 (3.3V)
- no-connect marks 1 -> 0
